File: electronics/Pico.kicad_sch (KiCad schematic)
At the start: 36 parts, among them J1 USB_B_Micro, J7 Conn_ARM_JTAG_SWD_10, J9 Conn_01x08, SW1 PTS645SK50SMTR92LFS, U1 STM32F415RGTx, U4 USBLC6-2SC6, Y2 Crystal_GND24

Commit message: Tweaked parts to use Basic parts which are cheaper.
Parts:
- C10, C11, C12, C17, C2, C5, C6, C7, C8, C9: JLCPCB C432917 -> C1525
- C3, C4: JLCPCB C696849 -> C1548
- C43, C46, C47: JLCPCB C76612 -> C23630
- D1: JLCPCB C2837377 -> C2286
- D10: JLCPCB C84267 -> C2286
- D11: JLCPCB C7420325 -> C8598
- R1: JLCPCB C423025 -> (none)
- R4, R9: JLCPCB C11702 -> (none)
Changed lines of the file:
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@@
 			)
 		)
-		(property "JLCPCB" "C432917"
+		(property "JLCPCB" "C1525"
 			(at 50.8 181.61 0)
 			(effects
@@
 			)
 		)
-		(property "JLCPCB" "C432917"
+		(property "JLCPCB" "C1525"
 			(at 95.25 181.61 0)
 			(effects
@@
 			)
 		)
-		(property "JLCPCB" "C84267"
+		(property "JLCPCB" "C2286"
 			(at 245.11 31.75 0)
 			(effects
@@
 			)
 		)
-		(property "JLCPCB" "C7420325"
+		(property "JLCPCB" "C8598"
 			(at 53.34 29.21 0)
 			(effects
@@
 			)
 		)
-		(property "JLCPCB" "C432917"
+		(property "JLCPCB" "C1525"
 			(at 106.68 181.61 0)
 			(effects
@@
 			)
 		)
-		(property "JLCPCB" "C432917"
+		(property "JLCPCB" "C1525"
 			(at 60.96 181.61 0)
 			(effects
@@
 			)
 		)
-		(property "JLCPCB" "C696849"
+		(property "JLCPCB" "C1548"
 			(at 82.55 86.36 0)
 			(effects
@@
 			)
 		)
-		(property "JLCPCB" "C432917"
+		(property "JLCPCB" "C1525"
 			(at 83.82 181.61 0)
 			(effects
@@
 			)
 		)
-		(property "JLCPCB" "C432917"
+		(property "JLCPCB" "C1525"
 			(at 40.64 181.61 0)
 			(effects
@@
 			)
 		)
-		(property "JLCPCB" "C432917"
+		(property "JLCPCB" "C1525"
 			(at 77.47 138.43 0)
 			(effects
@@
 			)
 		)
-		(property "JLCPCB" "C432917"
+		(property "JLCPCB" "C1525"
 			(at 30.48 181.61 0)
 			(effects
@@
 			)
 		)
-		(property "JLCPCB" "C432917"
+		(property "JLCPCB" "C1525"
 			(at 118.11 181.61 0)
 			(effects
@@
 			)
 		)
-		(property "JLCPCB" "C423025"
+		(property "JLCPCB" ""
 			(at 34.29 48.26 0)
 			(effects
@@
 			)
 		)
-		(property "JLCPCB" "C76612"
+		(property "JLCPCB" "C23630"
 			(at 44.45 44.45 0)
 			(effects
@@
 			)
 		)
-		(property "JLCPCB" "C11702"
+		(property "JLCPCB" ""
 			(at 107.95 74.93 0)
 			(effects
@@
 			)
 		)
-		(property "JLCPCB" "C76612"
+		(property "JLCPCB" "C23630"
 			(at 124.46 137.16 0)
 			(effects
@@
 			)
 		)
-		(property "JLCPCB" "C696849"
+		(property "JLCPCB" "C1548"
 			(at 82.55 72.39 0)
 			(effects
@@
 			)
 		)
-		(property "JLCPCB" "C432917"
+		(property "JLCPCB" "C1525"
 			(at 72.39 181.61 0)
 			(effects
@@
 			)
 		)
-		(property "JLCPCB" "C11702"
+		(property "JLCPCB" ""
 			(at 67.31 113.03 0)
 			(effects
@@
 			)
 		)
-		(property "JLCPCB" "C76612"
+		(property "JLCPCB" "C23630"
 			(at 113.03 137.16 0)
 			(effects
@@
 			)
 		)
-		(property "JLCPCB" "C2837377"
+		(property "JLCPCB" "C2286"
 			(at 245.11 22.86 0)
 			(effects

Commit message: Ordered this version.
Parts:
- SW1: footprint footprints:SW4_PTS645SK50SMTR92LFS_CNK -> footprints:PTS645SK50SMTR92LFS_CNK
Connections:
- net DISP_SO is gone; now on net DISP_DATA: U1.22 (PA6)
- net BOOT: now also U1.56 (PB4)
- net DISP_DATA: no longer U1.23 (PA7)
- new net DISP_SI: U1.23 (PA7)
Changed lines of the file:
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@@
 	(wire
 		(pts
-			(xy 107.95 67.31) (xy 134.62 67.31)
+			(xy 125.73 67.31) (xy 134.62 67.31)
 		)
 		(stroke
@@
 	(wire
 		(pts
+			(xy 170.18 115.57) (xy 177.8 115.57)
+		)
+		(stroke
+			(width 0)
+			(type default)
+		)
+	)
+	(wire
+		(pts
 			(xy 50.8 175.26) (xy 60.96 175.26)
 		)
@@
 		)
 	)
-	(label "BOOT"
-		(at 76.2 129.54 180)
-		(fields_autoplaced yes)
-		(effects
-			(font
-				(size 1.27 1.27)
-			)
-			(justify right bottom)
-		)
-	)
 	(label "OSC_IN"
 		(at 100.33 72.39 180)
@@
 		)
 	)
-	(label "BOOT"
-		(at 107.95 67.31 0)
+	(label "OSC_OUT"
+		(at 100.33 86.36 180)
 		(fields_autoplaced yes)
 		(effects
@@
 				(size 1.27 1.27)
 			)
-			(justify left bottom)
+			(justify right bottom)
 		)
 	)
-	(label "OSC_OUT"
-		(at 100.33 86.36 180)
+	(label "LED2"
+		(at 228.6 31.75 0)
 		(fields_autoplaced yes)
 		(effects
@@
 				(size 1.27 1.27)
 			)
-			(justify right bottom)
+			(justify left bottom)
 		)
 	)
-	(label "LED2"
-		(at 228.6 31.75 0)
+	(global_label "BOOT"
+		(shape input)
+		(at 76.2 129.54 0)
 		(fields_autoplaced yes)
 		(effects
@@
 				(size 1.27 1.27)
 			)
-			(justify left bottom)
+			(justify left)
+		)
+		(property "Intersheetrefs" "${INTERSHEET_REFS}"
+			(at 84.0838 129.54 0)
+			(effects
+				(font
+					(size 1.27 1.27)
+				)
+				(justify left)
+				(hide yes)
+			)
 		)
 	)
@@
 		)
 	)
-	(global_label "DISP_SO"
+	(global_label "DISP_SI"
 		(shape input)
-		(at 177.8 77.47 0)
+		(at 177.8 80.01 0)
 		(fields_autoplaced yes)
 		(effects
@@
 		)
 		(property "Intersheetrefs" "${INTERSHEET_REFS}"
-			(at 188.6471 77.47 0)
+			(at 187.9214 80.01 0)
 			(effects
 				(font
@@
 		)
 	)
+	(global_label "BOOT"
+		(shape input)
+		(at 125.73 67.31 180)
+		(fields_autoplaced yes)
+		(effects
+			(font
+				(size 1.27 1.27)
+			)
+			(justify right)
+		)
+		(property "Intersheetrefs" "${INTERSHEET_REFS}"
+			(at 117.8462 67.31 0)
+			(effects
+				(font
+					(size 1.27 1.27)
+				)
+				(justify right)
+				(hide yes)
+			)
+		)
+	)
 	(global_label "LED2"
 		(shape input)
@@
 		)
 	)
+	(global_label "BOOT"
+		(shape input)
+		(at 177.8 115.57 0)
+		(fields_autoplaced yes)
+		(effects
+			(font
+				(size 1.27 1.27)
+			)
+			(justify left)
+		)
+		(property "Intersheetrefs" "${INTERSHEET_REFS}"
+			(at 185.6838 115.57 0)
+			(effects
+				(font
+					(size 1.27 1.27)
+				)
+				(justify left)
+				(hide yes)
+			)
+		)
+	)
 	(global_label "LED1"
 		(shape input)
@@
 	(global_label "DISP_DATA"
 		(shape input)
-		(at 177.8 80.01 0)
+		(at 177.8 77.47 0)
 		(fields_autoplaced yes)
 		(effects
@@
 		)
 		(property "Intersheetrefs" "${INTERSHEET_REFS}"
-			(at 190.5219 80.01 0)
+			(at 190.5219 77.47 0)
 			(effects
 				(font
@@
 			)
 		)
-		(property "Footprint" "footprints:SW4_PTS645SK50SMTR92LFS_CNK"
+		(property "Footprint" "footprints:PTS645SK50SMTR92LFS_CNK"
 			(at 20.32 121.92 0)
 			(effects

Commit message: Updated parts based on request from JLCPCB.
Parts:
- J1: JLCPCB C2926986 -> C132562
Changed lines of the file:
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@@
 			)
 		)
-		(property "JLCPCB" "C2926986"
+		(property "JLCPCB" "C132562"
 			(at 21.59 34.29 0)
 			(effects

Commit message: Made some changes and thought I should check it in.
Other:
- note added: "These can be used for SPI2"
Changed lines of the file:
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@@
+		)
+	)
+	(text "These can be used for SPI2"
+		(exclude_from_sim no)
+		(at 202.946 139.7 0)
+		(effects
+			(font
+				(size 1.27 1.27)
+			)
 		)
 	)
