File: electronics/Can.kicad_sch (KiCad schematic)
At the start: 14 parts, among them J10 Conn_01x04, U2 TCAN1043xDxQ1

Commit message: Updated design to rev C
Parts:
- C13, C14: JLC (none) -> C1525; JLCPCB C1525 -> (none)
- C15, C16: JLC (none) -> C52923; JLCPCB C52923 -> (none)
- D12: JLC (none) -> C2105; JLCPCB C2105 -> (none)
- D4: JLC (none) -> C32677; JLCPCB C32677 -> (none)
- J10: JLC (none) -> C160354; JLCPCB C160354 -> (none); now not fitted
- R10: JLC (none) -> C25765; JLCPCB C93942 -> (none)
- R11, R20: JLC (none) -> C25744; JLCPCB C25744 -> (none)
- R12: JLC (none) -> C25079; JLCPCB C25079 -> (none)
- R19: value 100k -> 1K; JLC (none) -> C11702; JLCPCB C102750 -> (none)
- U2: JLC (none) -> C1848115; JLCPCB C1848115 -> (none)
Connections:
- net +12V: now also R20.1; no longer R19.1
- net GND: now also R19.2; no longer R20.2
- net VIN_MEAS: now also R19.1, R20.2; no longer R19.2, R20.1
Other:
- moved on the sheet: R19, R20
Changed lines of the file:
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@@
 (kicad_sch
-	(version 20231120)
+	(version 20250114)
 	(generator "eeschema")
-	(generator_version "8.0")
+	(generator_version "9.0")
 	(paper "A4")
 	(junction
@@
 			)
 		)
-		(property "JLCPCB" "C1848115"
+		(property "JLC" "C1848115"
 			(at 179.07 85.09 0)
 			(effects
@@
 			)
 		)
-		(property "JLCPCB" "C52923"
+		(property "JLC" "C52923"
 			(at 55.88 55.88 0)
 			(effects
@@
 			)
 		)
-		(property "JLCPCB" "C52923"
+		(property "JLC" "C52923"
 			(at 57.15 119.38 0)
 			(effects
@@
 	(symbol
 		(lib_id "Device:R")
+		(at 69.85 102.87 0)
+		(unit 1)
+		(exclude_from_sim no)
+		(in_bom yes)
+		(on_board yes)
+		(dnp no)
+		(fields_autoplaced yes)
+		(property "Reference" "R20"
+			(at 72.39 101.5999 0)
+			(effects
+				(font
+					(size 1.27 1.27)
+				)
+				(justify left)
+			)
+		)
+		(property "Value" "10k"
+			(at 72.39 104.1399 0)
+			(effects
+				(font
+					(size 1.27 1.27)
+				)
+				(justify left)
+			)
+		)
+		(property "Footprint" "Resistor_SMD:R_0402_1005Metric"
+			(at 68.072 102.87 90)
+			(effects
+				(font
+					(size 1.27 1.27)
+				)
+				(hide yes)
+			)
+		)
+		(property "Datasheet" "~"
+			(at 69.85 102.87 0)
+			(effects
+				(font
+					(size 1.27 1.27)
+				)
+				(hide yes)
+			)
+		)
+		(property "Description" ""
+			(at 69.85 102.87 0)
+			(effects
+				(font
+					(size 1.27 1.27)
+				)
+				(hide yes)
+			)
+		)
+		(property "JLC" "C25744"
+			(at 69.85 102.87 0)
+			(effects
+				(font
+					(size 1.27 1.27)
+				)
+				(hide yes)
+			)
+		)
+		(pin "2"
+		)
+		(pin "1"
+		)
+		(instances
+			(project "FRCMotorTester"
+				(path "/8b7d42f7-da13-4f9b-ae64-d2ea00a4933f/901daec7-ebc5-4b56-9f65-1aeb323e4fd0"
+					(reference "R20")
+					(unit 1)
+				)
+			)
+		)
+	)
+	(symbol
+		(lib_id "Device:R")
 		(at 69.85 119.38 0)
 		(unit 1)
@@
 		(dnp no)
 		(fields_autoplaced yes)
-		(property "Reference" "R20"
+		(property "Reference" "R19"
 			(at 72.39 118.1099 0)
 			(effects
@@
 			)
 		)
-		(property "Value" "10k"
+		(property "Value" "1K"
 			(at 72.39 120.6499 0)
 			(effects
@@
 			)
 		)
-		(property "JLCPCB" "C25744"
+		(property "JLC" "C11702"
 			(at 69.85 119.38 0)
-			(effects
-				(font
-					(size 1.27 1.27)
-				)
-				(hide yes)
-			)
-		)
-		(pin "2"
-		)
-		(pin "1"
-		)
-		(instances
-			(project "FRCMotorTester"
-				(path "/8b7d42f7-da13-4f9b-ae64-d2ea00a4933f/901daec7-ebc5-4b56-9f65-1aeb323e4fd0"
-					(reference "R20")
-					(unit 1)
-				)
-			)
-		)
-	)
-	(symbol
-		(lib_id "Device:R")
-		(at 69.85 102.87 0)
-		(unit 1)
-		(exclude_from_sim no)
-		(in_bom yes)
-		(on_board yes)
-		(dnp no)
-		(fields_autoplaced yes)
-		(property "Reference" "R19"
-			(at 72.39 101.5999 0)
-			(effects
-				(font
-					(size 1.27 1.27)
-				)
-				(justify left)
-			)
-		)
-		(property "Value" "100k"
-			(at 72.39 104.1399 0)
-			(effects
-				(font
-					(size 1.27 1.27)
-				)
-				(justify left)
-			)
-		)
-		(property "Footprint" "Resistor_SMD:R_0402_1005Metric"
-			(at 68.072 102.87 90)
-			(effects
-				(font
-					(size 1.27 1.27)
-				)
-				(hide yes)
-			)
-		)
-		(property "Datasheet" "~"
-			(at 69.85 102.87 0)
-			(effects
-				(font
-					(size 1.27 1.27)
-				)
-				(hide yes)
-			)
-		)
-		(property "Description" ""
-			(at 69.85 102.87 0)
-			(effects
-				(font
-					(size 1.27 1.27)
-				)
-				(hide yes)
-			)
-		)
-		(property "JLCPCB" "C102750"
-			(at 69.85 102.87 0)
 			(effects
 				(font
@@
 			)
 		)
-		(property "JLCPCB" "C1525"
+		(property "JLC" "C1525"
 			(at 162.56 31.75 0)
 			(effects
@@
 			)
 		)
-		(property "JLCPCB" "C25079"
+		(property "JLC" "C25079"
 			(at 239.395 83.82 0)
 			(effects
@@
 			)
 		)
-		(property "JLCPCB" "C2105"
-			(at 43.18 119.38 0)
+		(property "JLC" "C2105"
+			(at 43.18 119.38 90)
 			(effects
 				(font
@@
 		(in_bom yes)
 		(on_board yes)
-		(dnp no)
+		(dnp yes)
 		(fields_autoplaced yes)
 		(property "Reference" "J10"
@@
 			)
 		)
-		(property "JLCPCB" "C160354"
+		(property "Digikey" "455-1721-ND"
 			(at 270.51 85.09 0)
 			(effects
@@
 			)
 		)
-		(property "Digikey" "455-1721-ND"
+		(property "JLC" "C160354"
 			(at 270.51 85.09 0)
 			(effects
@@
 			)
 		)
-		(property "JLCPCB" "C93942"
+		(property "JLC" "C25765"
 			(at 68.58 39.37 0)
 			(effects
@@
 			)
 		)
-		(property "JLCPCB" "C32677"
+		(property "JLC" "C32677"
 			(at 217.17 96.52 0)
 			(effects
@@
 			)
 		)
-		(property "JLCPCB" "C25744"
+		(property "JLC" "C25744"
 			(at 68.58 55.88 0)
 			(effects
@@
 			)
 		)
-		(property "JLCPCB" "C1525"
+		(property "JLC" "C1525"
 			(at 162.56 54.61 0)
 			(effects
