File: electronics/FRCMotorTester.kicad_pcb (KiCad board)
At the start: 4 copper layers, 85.6 x 70.8 mm, 99 parts, among them J1 USB_B_Micro, J10 Conn_01x04, J2 Conn_01x02_Socket, J3 Conn_01x06, J7 Conn_ARM_JTAG_SWD_10, J9 Conn_01x08, Q2 IRLML6401, SW1 PTS645SK50SMTR92LFS, SW2 RotaryEncoder_Switch, SW3 RotaryEncoder_Switch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

Commit message: Updated design to rev C
Parts:
- removed C25, C27: 10u, Capacitor_SMD:C_0805_2012Metric
- removed J7: Conn_ARM_JTAG_SWD_10, Connector:Tag-Connect_TC2050-IDC-NL_2x05_P1.27mm_Vertical_with_bottom_clip
- removed JP1: Jumper_NO_Small, Jumper:SolderJumper-2_P1.3mm_Open_TrianglePad1.0x1.5mm
- removed Q2: IRLML6401, Package_TO_SOT_SMD:SOT-23
- removed R13: 1.6k, Resistor_SMD:R_0402_1005Metric
- removed R14, R16: 1k, Resistor_SMD:R_0402_1005Metric
- removed R15: 1.3k, Resistor_SMD:R_0402_1005Metric
- removed TP9: TestPoint, TestPoint:TestPoint_Pad_D1.0mm
- removed U5, U7: LM1117DT-ADJ, Package_TO_SOT_SMD:SOT-223-3_TabPin2
- added D7: D_Schottky, Diode_SMD:D_SOD-123, F.Cu at (124.8, 40.8)
- added J4: Conn_ARM_SWD_TagConnect_TC2030-NL, Connector:Tag-Connect_TC2030-IDC-NL_2x03_P1.27mm_Vertical, F.Cu at (141.4, 103.1)
- added U1: AMS1117-3.3, Package_TO_SOT_SMD:SOT-223-3_TabPin2, F.Cu at (132.2, 61.0)
- R1, R2, R3: footprint Resistor_SMD:R_0402_1005Metric -> Resistor_SMD:R_0603_1608Metric
- R17: value 49.9k -> 47K; footprint Resistor_SMD:R_0402_1005Metric -> Resistor_SMD:R_0603_1608Metric
- R18: value 9.53k -> 9.1K; footprint Resistor_SMD:R_0402_1005Metric -> Resistor_SMD:R_0603_1608Metric
- R19: value 100k -> 1K
- moved C23 16.9 mm to (140.5, 61.1), turned to 0 degrees
- moved TP8 16.1 mm to (139.4, 57.9)
- moved C22 11.7 mm to (125.2, 63.4), turned to 180 degrees
- moved TP7 6.38 mm to (127.9, 51.2)
- moved R3 1.01 mm to (126.1, 78.0)
- moved R20 0.85 mm to (109.1, 49.7), turned to 90 degrees
- moved R19 0.76 mm to (109.1, 47.2), turned to 90 degrees
Connections:
- DS1 pad A: 3V0 -> 3V3
- R19 pad 1: +12V -> VIN_MEAS
- R19 pad 2: VIN_MEAS -> GND
- R20 pad 1: VIN_MEAS -> +12V
- R20 pad 2: GND -> VIN_MEAS
Routing:
- net 3V0: track 31.7 -> 0.00 mm
- net 3V3: track 54.0 -> 68.5 mm, vias 28 -> 25
- net Net-(U7-ADJ): track 7.36 -> 0.00 mm
- net Net-(U5-ADJ): track 7.30 -> 0.00 mm
- net GND: track 77.4 -> 70.8 mm, vias 56 -> 53
- net /Power/VIN: track 22.2 -> 16.7 mm
- net SWDIO: track 24.6 -> 19.5 mm, vias 2 -> 0
- net VIN_MEAS: track 65.7 -> 69.9 mm
- net NRST: track 44.0 -> 47.2 mm
- net +12V: track 51.2 -> 48.4 mm
- net Net-(U3-PB1): track 6.66 -> 5.89 mm
Other:
- board text added: "Team 4360 and 7048 Brushless Buddy Rev C 2026"
- board text removed: "DISP SO SCLK DATA RESET SS"
- board text removed: "Team 4360 and 7048 Brushless Buddy Rev B 2024"
