File: electronics/IO.kicad_sch (KiCad schematic)
At the start: 25 parts, among them J3 Conn_01x06, SW1 RotaryEncoder_Switch, SW2 RotaryEncoder_Switch

Commit message: Updated design to rev C
Parts:
- C29: renamed from C1; JLC (none) -> C15195; JLCPCB C15195 -> (none)
- C30: renamed from C3; JLC (none) -> C15195; JLCPCB C15195 -> (none)
- C31: renamed from C7; JLC (none) -> C1525; JLCPCB C1525 -> (none)
- C32: renamed from C2; JLC (none) -> C15195; JLCPCB C15195 -> (none)
- C33: renamed from C4; JLC (none) -> C15195; JLCPCB C15195 -> (none)
- C34: renamed from C8; JLC (none) -> C1525; JLCPCB C1525 -> (none)
- C35, C36, C37, C38, C39: JLC (none) -> C52923; JLCPCB C52923 -> (none)
- C40, C41, C42: JLC (none) -> C23630; JLCPCB C23630 -> (none)
- D5, D6: JLC (none) -> C32677; JLCPCB C32677 -> (none)
- DS1: now not fitted
- J3: JLC (none) -> C471518; JLCPCB C471518 -> (none); now not fitted
- renumbered SW1 to SW2, SW2 to SW3
Connections:
- net 3V0 is gone; now on net +3.3V: DS1.A (LED+)
Changed lines of the file:
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@@
 (kicad_sch
-	(version 20231120)
+	(version 20250114)
 	(generator "eeschema")
-	(generator_version "8.0")
+	(generator_version "9.0")
 	(paper "A4")
+	(text "New Haven OLED\nNHD-C12832A1Z-FSW-FBW-3V3\n"
+		(exclude_from_sim no)
+		(at 236.22 63.5 0)
+		(effects
+			(font
+				(size 1.27 1.27)
+			)
+			(justify left bottom)
+		)
+	)
 	(junction
 		(at 77.47 44.45)
@@
 		)
 	)
-	(text "New Haven OLED\nNHD-C12832A1Z-FSW-FBW-3V3\n"
-		(exclude_from_sim no)
-		(at 236.22 63.5 0)
-		(effects
-			(font
-				(size 1.27 1.27)
-			)
-			(justify left bottom)
-		)
-	)
-	(global_label "3V0"
-		(shape input)
-		(at 200.66 119.38 0)
-		(fields_autoplaced yes)
-		(effects
-			(font
-				(size 1.27 1.27)
-			)
-			(justify left)
-		)
-		(property "Intersheetrefs" "${INTERSHEET_REFS}"
-			(at 207.1528 119.38 0)
-			(effects
-				(font
-					(size 1.27 1.27)
-				)
-				(justify left)
-				(hide yes)
-			)
-		)
-	)
 	(global_label "ENC1B"
 		(shape input)
@@
 		(dnp no)
 		(fields_autoplaced yes)
-		(property "Reference" "C3"
+		(property "Reference" "C30"
 			(at 45.72 39.3699 0)
 			(effects
@@
 			)
 		)
-		(property "JLCPCB" "C15195"
+		(property "JLC" "C15195"
 			(at 41.91 40.64 0)
 			(effects
@@
 			)
 		)
-		(property "JLCPCB" "C23630"
-			(at 218.44 106.68 0)
+		(property "JLC" "C23630"
+			(at 218.44 106.68 90)
 			(effects
 				(font
@@
 		(in_bom yes)
 		(on_board yes)
-		(dnp no)
+		(dnp yes)
 		(fields_autoplaced yes)
 		(property "Reference" "J3"
@@
 			)
 		)
-		(property "JLCPCB" "C471518"
+		(property "Digikey" "455-1723-ND"
 			(at 91.44 86.36 0)
 			(effects
@@
 			)
 		)
-		(property "Digikey" "455-1723-ND"
+		(property "JLC" "C471518"
 			(at 91.44 86.36 0)
 			(effects
@@
 			)
 		)
-		(property "JLCPCB" "C52923"
-			(at 254 128.27 0)
+		(property "JLC" "C52923"
+			(at 254 128.27 90)
 			(effects
 				(font
@@
 	)
 	(symbol
+		(lib_id "power:+3.3V")
+		(at 200.66 119.38 0)
+		(unit 1)
+		(exclude_from_sim no)
+		(in_bom yes)
+		(on_board yes)
+		(dnp no)
+		(fields_autoplaced yes)
+		(property "Reference" "#PWR022"
+			(at 200.66 123.19 0)
+			(effects
+				(font
+					(size 1.27 1.27)
+				)
+				(hide yes)
+			)
+		)
+		(property "Value" "+3.3V"
+			(at 200.66 114.3 0)
+			(effects
+				(font
+					(size 1.27 1.27)
+				)
+			)
+		)
+		(property "Footprint" ""
+			(at 200.66 119.38 0)
+			(effects
+				(font
+					(size 1.27 1.27)
+				)
+				(hide yes)
+			)
+		)
+		(property "Datasheet" ""
+			(at 200.66 119.38 0)
+			(effects
+				(font
+					(size 1.27 1.27)
+				)
+				(hide yes)
+			)
+		)
+		(property "Description" ""
+			(at 200.66 119.38 0)
+			(effects
+				(font
+					(size 1.27 1.27)
+				)
+				(hide yes)
+			)
+		)
+		(pin "1"
+		)
+		(instances
+			(project "FRCMotorTester"
+				(path "/8b7d42f7-da13-4f9b-ae64-d2ea00a4933f/8ce18279-c24a-4fc6-a071-ab76dabc1fca"
+					(reference "#PWR022")
+					(unit 1)
+				)
+			)
+		)
+	)
+	(symbol
 		(lib_id "power:GND")
 		(at 77.47 45.72 0)
@@
 		(dnp no)
 		(fields_autoplaced yes)
-		(property "Reference" "#PWR05"
+		(property "Reference" "#PWR040"
 			(at 77.47 52.07 0)
 			(effects
@@
 			)
 		)
-		(property "JLCPCB" "C32677"
+		(property "JLC" "C32677"
 			(at 59.69 130.81 0)
 			(effects
@@
 		(dnp no)
 		(fields_autoplaced yes)
-		(property "Reference" "C8"
+		(property "Reference" "C34"
 			(at 180.34 38.1 0)
 			(effects
@@
 			)
 		)
-		(property "JLCPCB" "C1525"
+		(property "JLC" "C1525"
 			(at 176.53 39.37 0)
 			(effects
@@
 		(on_board yes)
 		(dnp no)
-		(property "Reference" "C1"
+		(property "Reference" "C29"
 			(at 34.29 39.37 0)
 			(effects
@@
 			)
 		)
-		(property "JLCPCB" "C15195"
+		(property "JLC" "C15195"
 			(at 30.48 40.64 0)
 			(effects
@@
 			)
 		)
-		(property "JLCPCB" "C32677"
+		(property "JLC" "C32677"
 			(at 43.18 130.81 0)
 			(effects
@@
 		(dnp no)
 		(fields_autoplaced yes)
-		(property "Reference" "C4"
+		(property "Reference" "C33"
 			(at 138.43 39.3699 0)
 			(effects
@@
 			)
 		)
-		(property "JLCPCB" "C15195"
+		(property "JLC" "C15195"
 			(at 134.62 40.64 0)
 			(effects
@@
 		(dnp no)
 		(fields_autoplaced yes)
-		(property "Reference" "#PWR06"
+		(property "Reference" "#PWR042"
 			(at 170.18 52.07 0)
 			(effects
@@
 			)
 		)
-		(property "JLCPCB" "C52923"
-			(at 238.76 128.27 0)
+		(property "JLC" "C52923"
+			(at 238.76 128.27 90)
 			(effects
 				(font
@@
 			)
 		)
-		(property "JLCPCB" "C23630"
-			(at 218.44 119.38 0)
+		(property "JLC" "C23630"
+			(at 218.44 119.38 90)
 			(effects
 				(font
@@
 		(dnp yes)
 		(fields_autoplaced yes)
-		(property "Reference" "SW1"
+		(property "Reference" "SW2"
 			(at 60.96 20.32 0)
 			(effects
@@
 			)
 		)
-		(property "JLCPCB" ""
-			(at 60.96 30.48 0)
-			(effects
-				(font
-					(size 1.27 1.27)
-				)
-				(hide yes)
-			)
-		)
 		(property "Digikey" "PEC11R-4220K-S0024-ND"
 			(at 60.96 30.48 0)
@@
 		(dnp no)
 		(fields_autoplaced yes)
-		(property "Reference" "#PWR03"
+		(property "Reference" "#PWR039"
 			(at 44.45 55.88 0)
 			(effects
@@
 		(on_board yes)
 		(dnp no)
-		(property "Reference" "C7"
+		(property "Reference" "C31"
 			(at 87.63 38.1 0)
 			(effects
@@
 			)
 		)
-		(property "JLCPCB" "C1525"
+		(property "JLC" "C1525"
 			(at 83.82 39.37 0)
 			(effects
@@
 		(on_board yes)
 		(dnp no)
-		(property "Reference" "C2"
+		(property "Reference" "C32"
 			(at 127 39.37 0)
 			(effects
@@
 			)
 		)
-		(property "JLCPCB" "C15195"
+		(property "JLC" "C15195"
 			(at 123.19 40.64 0)
 			(effects
@@
 		(dnp no)
 		(fields_autoplaced yes)
-		(property "Reference" "#PWR04"
+		(property "Reference" "#PWR041"
 			(at 137.16 55.88 0)
 			(effects
@@
 		(dnp yes)
 		(fields_autoplaced yes)
-		(property "Reference" "SW2"
+		(property "Reference" "SW3"
 			(at 153.67 20.32 0)
 			(effects
@@
 			)
 		)
-		(property "JLCPCB" ""
-			(at 153.67 30.48 0)
-			(effects
-				(font
-					(size 1.27 1.27)
-				)
-				(hide yes)
-			)
-		)
 		(property "Digikey" "PEC11R-4220K-S0024-ND"
 			(at 153.67 30.48 0)
@@
 			)
 		)
-		(property "JLCPCB" "C52923"
-			(at 261.62 128.27 0)
+		(property "JLC" "C52923"
+			(at 261.62 128.27 90)
 			(effects
 				(font
@@
 			)
 		)
-		(property "JLCPCB" "C52923"
-			(at 246.38 128.27 0)
+		(property "JLC" "C52923"
+			(at 246.38 128.27 90)
 			(effects
 				(font
@@
 			)
 		)
-		(property "JLCPCB" "C23630"
-			(at 229.87 128.27 0)
+		(property "JLC" "C23630"
+			(at 229.87 128.27 90)
 			(effects
 				(font
@@
 			)
 		)
-		(property "JLCPCB" "C52923"
-			(at 269.24 128.27 0)
+		(property "JLC" "C52923"
+			(at 269.24 128.27 90)
 			(effects
 				(font
@@
 		(in_bom yes)
 		(on_board yes)
-		(dnp no)
+		(dnp yes)
 		(fields_autoplaced yes)
 		(property "Reference" "DS1"
