File: electronics/Power.kicad_sch (KiCad schematic)
At the start: 25 parts, among them J2 Conn_01x02_Socket, Q2 IRLML6401, U10 AOZ1280CI, U5 LM1117DT-ADJ, U7 LM1117DT-ADJ

Commit message: Updated design to rev C
Parts:
- removed C25, C27: 10u, Capacitor_SMD:C_0805_2012Metric, symbol Device:C
- removed JP1: Jumper_NO_Small, Jumper:SolderJumper-2_P1.3mm_Open_TrianglePad1.0x1.5mm, symbol Device:Jumper_NO_Small
- removed Q2: IRLML6401, Package_TO_SOT_SMD:SOT-23, symbol Transistor_FET:IRLML6401
- removed R13: 1.6k, Resistor_SMD:R_0402_1005Metric, symbol Device:R
- removed R14, R16: 1k, Resistor_SMD:R_0402_1005Metric, symbol Device:R
- removed R15: 1.3k, Resistor_SMD:R_0402_1005Metric, symbol Device:R
- removed TP9: TestPoint, TestPoint:TestPoint_Pad_D1.0mm, symbol Connector:TestPoint
- removed U5, U7: LM1117DT-ADJ, Package_TO_SOT_SMD:SOT-223-3_TabPin2, symbol Regulator_Linear:LM1117DT-ADJ
- added D7: D_Schottky, Diode_SMD:D_SOD-123, symbol Device:D_Schottky
- added U1: AMS1117-3.3, Package_TO_SOT_SMD:SOT-223-3_TabPin2, symbol Regulator_Linear:AMS1117-3.3
- C22, C23: JLC (none) -> C15850; JLCPCB C15850 -> (none)
- C24: renamed from C10; JLC (none) -> C15850; JLCPCB C15850 -> (none)
- C26: renamed from C11; JLC (none) -> C15195; JLCPCB C15195 -> (none)
- C28: renamed from C12; JLC (none) -> C15850; JLCPCB C15850 -> (none)
- D2: renamed from D1; JLC (none) -> C8598; JLCPCB C8598 -> (none)
- D3: renamed from D22; JLC (none) -> C8598; JLCPCB C8598 -> (none)
- J2: JLC (none) -> C173752; JLCPCB C173752 -> (none); now not fitted
- L1: JLC (none) -> C1330201; JLCPCB C1330201 -> (none)
- R17: renamed from R9; value 49.9k -> 47K; footprint Resistor_SMD:R_0402_1005Metric -> Resistor_SMD:R_0603_1608Metric; JLC (none) -> C25819; JLCPCB C100457 -> (none)
- R18: renamed from R10; value 9.53k -> 9.1K; footprint Resistor_SMD:R_0402_1005Metric -> Resistor_SMD:R_0603_1608Metric; JLC (none) -> C23260; JLCPCB C103191 -> (none)
- U6: renamed from U10; JLC (none) -> C41240; JLCPCB C41240 -> (none)
Connections:
- net +12V: now also D7.1 (K)
- net 3V3: now also U1.2 (VO)
- net GND: now also U1.1 (GND)
- net VCC: now also U1.3 (VI)
- net VIN: now also D7.2 (A)
